File: PCB/Companion_totem_TP/Companion_totem_TP.kicad_pcb (KiCad board)
At the start: 2 copper layers, 258.7 x 94.4 mm, 128 parts, among them J1 Conn_01x02_Socket, J2 Conn_01x02_Socket, U1 xiao-ble, U2 xiao-ble

Commit message: Added TP, Split L&R
Parts:
- removed the REF** at (187.8, 100.0)
- removed the REF** at (178.8, 72.5)
- removed the REF** at (196.8, 72.5)
- added J4: Red_mouse_stick, TOTEMlib:T460S_TP, F.Cu at (187.8, 72.5)
- added J5: Trackpoint module, TOTEMlib:TP_input, B.Cu at (219.3, 101.3)
- added J5: Trackpoint module, TOTEMlib:TP_input, B.Cu at (219.3, 104.5)
- added Trackpoint_in: Trackpoint module, Connector_PinSocket_2.54mm:PinSocket_1x05_P2.54mm_Vertical, F.Cu at (170.3, 106.1)
- moved J3 67.6 mm to (173.3, 106.1), turned to 0 degrees
- moved R2 23.0 mm to (219.5, 100.2), turned to 0 degrees
- moved C1 20.3 mm to (219.5, 102.2), turned to 0 degrees
- moved R1 17.6 mm to (219.5, 104.2), turned to 180 degrees
- moved R3 14.9 mm to (219.5, 106.2), turned to 0 degrees
- moved JP1 12.5 mm to (219.4, 107.7), turned to 180 degrees
- moved G*** 1.00 mm to (215.0, 110.1)
- moved G*** 1.00 mm to (220.5, 110.1)
- turned SWL16 to -80 degrees
- turned SWR16 to 80 degrees
- renumbered Trackpoint_in to J3
Connections:
- ENCR17 pad : (no net) -> COL2_R
- ENCR17 pad 1: (no net) -> COL2_R
- ENCR17 pad 2: (no net) -> COL2_R
- U2 pad 7: unconnected-(U2-P1.11_TX_D6-Pad7) -> ENC_B_R
Routing:
- net TP_SCL: track 93.4 -> 159.5 mm
- net TP_4: track 0.00 -> 63.7 mm, vias 0 -> 2
- net VCC_R: track 71.5 -> 134.6 mm
- net TP_SDA: track 82.5 -> 143.8 mm
- net TP_2: track 0.00 -> 54.3 mm
- net TP_1: track 0.00 -> 52.3 mm, vias 0 -> 2
- net TP_3: track 0.00 -> 46.0 mm
- net Net-(J3-Pin_3): track 16.2 -> 59.4 mm
- net Net-(DR16-A): track 32.0 -> 3.35 mm, vias 3 -> 1
- net COL4_R: track 237.1 -> 215.7 mm
- net COL0_L: track 83.0 -> 65.8 mm
- net Net-(DL16-A): track 7.01 -> 22.4 mm
- net ROW2_R: track 287.3 -> 298.6 mm, vias 8 -> 7
- net COL0_R: track 116.3 -> 105.7 mm
- net COL2_R: track 182.5 -> 189.1 mm, vias 1 -> 4
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Other:
- outline, holes or cut-outs redrawn
- board text added: "T440 (Blue board)"
- board text added: "T460S (RED board)"
